File: PCB/board_test (copy1)/board_test.sch (KiCad schematic (older format))
At the start: 161 parts, among them J1 USB_A, J10 Conn_01x02_Female, J11 Conn_01x03_Male, J12 Conn_01x03_Male, J13 Conn_01x03_Male, J14 Conn_01x03_Male, J15 Conn_01x02_Female, J2 Conn_02x06_Top_Bottom, J3 Conn_02x06_Top_Bottom, J4 Conn_02x06_Top_Bottom, J5 Conn_02x06_Top_Bottom, J6 Conn_02x06_Top_Bottom, J7 Conn_02x06_Top_Bottom, J8 Conn_01x02_Female, J9 Conn_01x02_Female, U1 TMUX1119, U10 LTC2245, U11 RenzoChip, U2 TMUX1119, U3 LT1763, U4 LT1763, U5 NCP164ASN180T1G, U6 LTC1983-3, U7 LTC1983-3, U8 NCP164ASN180T1G, U9 SN74AUC2G06

Commit message: Vivado project added
Parts:
- removed J11, J12, J13, J14: Conn_01x03_Male, Connector_Coaxial:BNC_Win_364A2x95_Horizontal, symbol Connector:Conn_01x03_Male
- added J11, J12, J13, J14: Conn_01x02_Male, Connector_Coaxial:BNC_Amphenol_B6252HB-NPP3G-50_Horizontal, symbol Connector:Conn_01x02_Male
- added R1, R2, R3, R31, R32, R4: R_US, Resistor_SMD:R_0603_1608Metric, symbol Device:R_US
- C1, C10, C11, C14, C2, C30, C34: footprint Capacitor_SMD:C_0201_0603Metric -> Capacitor_SMD:C_0402_1005Metric
- C12, C52: footprint Capacitor_SMD:C_1206_3216Metric_Pad1.42x1.75mm_HandSolder -> Capacitor_SMD:C_0603_1608Metric
- C13, C15, C16, C17, C18, C20, C21, C24, C25, C26, C28, C29, C39, C50, C51, C53, C54, C6, C7, C8, C9: footprint Capacitor_SMD:C_0201_0603Metric -> Capacitor_SMD:C_0603_1608Metric
- C23: footprint Capacitor_SMD:C_0805_2012Metric_Pad1.15x1.40mm_HandSolder -> Capacitor_SMD:C_0201_0603Metric
- C3, C5: footprint Capacitor_SMD:CP_Elec_4x3 -> Capacitor_SMD:CP_Elec_5x3.9
- C31, C32, C33: footprint Capacitor_SMD:C_0201_0603Metric -> Capacitor_SMD:C_0603_1608Metric_Pad1.05x0.95mm_HandSolder
- C4: value 1uF -> 0.01uF; footprint Capacitor_SMD:C_0201_0603Metric -> Capacitor_SMD:C_0603_1608Metric
- C40, C41, C42, C43, C44, C45, C46, C47, C48, C49, C55: footprint Capacitor_SMD:C_0603_1608Metric_Pad1.05x0.95mm_HandSolder -> Capacitor_SMD:C_0603_1608Metric
- MUX1: footprint Package_SO:TSSOP-16_4.4x5mm_P0.65mm -> Package_SO:SOIC-16_3.9x9.9mm_P1.27mm
- OPAM1, OPAM2, OPAM3, OPAM4: footprint Package_SO:SSOP-8_2.95x2.8mm_P0.65mm -> Package_SO:SO-8_3.9x4.9mm_P1.27mm
- TP1, TP2, TP3, TP4, TP5, TP6, TP7, TP8: footprint Connector_PinHeader_2.00mm:PinHeader_1x01_P2.00mm_Vertical -> Connector_Pin:Pin_D1.4mm_L8.5mm_W2.8mm_FlatFork
- U1, U2: footprint Package_TO_SOT_SMD:SOT-23-6_Handsoldering -> Package_TO_SOT_SMD:SOT-363_SC-70-6_Handsoldering
Connections:
- net labels added: chip_clk18, chip_data_in18, chip_rst18
- wire segments 240 -> 250
